File: PCB/j201-board-v1/j201-board-v1.kicad_pcb (KiCad board)
At the start: 2 copper layers, 15.5 x 15.5 mm, 9 parts, among them J1 power (3V) [9V], J2 input (piezo), J3 output (jack), Q1 NJFET

Commit message: board design
Parts:
- Q1: value NJFET -> J201; footprint Package_TO_SOT_SMD:SOT-23 -> Package_TO_SOT_SMD:SOT-23-3
- moved C1 53.9 mm to (104.9, 58.7)
- moved J1 53.9 mm to (101.9, 59.2)
- moved R2 53.9 mm to (102.8, 54.9)
- moved R3 53.9 mm to (104.9, 54.9)
- moved J3 53.9 mm to (107.7, 54.6)
- moved J2 53.7 mm to (96.3, 54.6)
- moved Q1 53.5 mm to (99.8, 55.1), turned to 90 degrees
- moved C2 53.1 mm to (104.9, 52.1)
- moved R1 52.2 mm to (101.2, 52.1)
Routing:
- net /GND: track 39.9 -> 29.5 mm, vias 5 -> 3
- net /V+: track 7.56 -> 6.39 mm
- net Net-(J2-Pin_1): track 8.02 -> 6.90 mm
- net Net-(Q1-D): track 4.66 -> 5.39 mm
- net (no net): vias 1 -> 0
- added copper zone on F.Cu, net (none)
Other:
- board size 15.5 x 15.5 mm -> 20 x 20 mm
- board text added: "15mil"
