File: PCB/j201-board-v1/j201-board-v1.kicad_sch (KiCad schematic)
At the start: 9 parts, among them J1 input (piezo), J2 power (3V) [9V], J3 output (jack), Q1 NJFET

Commit message: update footprints
Parts:
- C1, C2: footprint (none) -> Capacitor_SMD:C_0805_2012Metric
- J1, J2, J3: footprint (none) -> !connections:P2
- Q1: footprint (none) -> Package_TO_SOT_SMD:SOT-23
- R1, R2, R3: footprint (none) -> Resistor_SMD:R_0805_2012Metric
Connections:
- net at J1.1 (Pin_1), R2.1: now also Q1.3 (G); no longer Q1.2 (G)
- net at C1.2, J1.2 (Pin_2), J2.2 (Pin_2)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: now also Q1.1 (S); no longer Q1.3 (S)
- net at C2.1, R1.2: now also Q1.2 (D); no longer Q1.1 (D)
Changed lines of the file:
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@@
       (effects (font (size 1.27 1.27)) (justify left))
     )
-    (property "Footprint" "" (at 112.522 113.03 90)
+    (property "Footprint" "Resistor_SMD:R_0805_2012Metric" (at 112.522 113.03 90)
       (effects (font (size 1.27 1.27)) hide)
     )
@@
       (effects (font (size 1.27 1.27)) (justify left))
     )
-    (property "Footprint" "" (at 128.27 97.79 0)
+    (property "Footprint" "Package_TO_SOT_SMD:SOT-23" (at 128.27 97.79 0)
       (effects (font (size 1.27 1.27)) hide)
     )
@@
       (effects (font (size 1.27 1.27)))
     )
-    (property "Footprint" "" (at 72.39 76.2 0)
+    (property "Footprint" "!connections:P2" (at 72.39 76.2 0)
       (effects (font (size 1.27 1.27)) hide)
     )
@@
       (effects (font (size 1.27 1.27)) (justify left))
     )
-    (property "Footprint" "" (at 89.8652 87.63 0)
+    (property "Footprint" "Capacitor_SMD:C_0805_2012Metric" (at 89.8652 87.63 0)
       (effects (font (size 1.27 1.27)) hide)
     )
@@
       (effects (font (size 1.27 1.27)) (justify left))
     )
-    (property "Footprint" "" (at 152.908 113.03 90)
+    (property "Footprint" "Resistor_SMD:R_0805_2012Metric" (at 152.908 113.03 90)
       (effects (font (size 1.27 1.27)) hide)
     )
@@
       (effects (font (size 1.27 1.27)))
     )
-    (property "Footprint" "" (at 144.78 90.4748 0)
+    (property "Footprint" "Capacitor_SMD:C_0805_2012Metric" (at 144.78 90.4748 0)
       (effects (font (size 1.27 1.27)) hide)
     )
@@
       (effects (font (size 1.27 1.27)))
     )
-    (property "Footprint" "" (at 168.91 91.44 0)
+    (property "Footprint" "!connections:P2" (at 168.91 91.44 0)
       (effects (font (size 1.27 1.27)) hide)
     )
@@
       (effects (font (size 1.27 1.27)) (justify left))
     )
-    (property "Footprint" "" (at 127.508 83.82 90)
+    (property "Footprint" "Resistor_SMD:R_0805_2012Metric" (at 127.508 83.82 90)
       (effects (font (size 1.27 1.27)) hide)
     )
@@
       (effects (font (size 1.27 1.27)))
     )
-    (property "Footprint" "" (at 99.06 100.33 0)
-      (effects (font (size 1.27 1.27)) hide)
-    )
+    (property "Footprint" "!connections:P2" (at 99.06 100.33 0)
+      (effects (font (size 1.27 1.27)) hide)
+    )

Commit message: board v1
Parts:
- renumbered J2 to J1, J1 to J2, R2 to R1, R1 to R2
Connections:
- net GND: now reaches C1.2, J1.2 (Pin_2), J2.2 (Pin_2), J3.2 (Pin_2), Q1.1 (S), R1.2, R3.2
- net V+: now reaches C1.1, J1.1 (Pin_1), R2.1

Commit message: board design
Parts:
- Q1: value NJFET -> J201; footprint Package_TO_SOT_SMD:SOT-23 -> Package_TO_SOT_SMD:SOT-23-3
Changed lines of the file:
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@@
       (effects (font (size 1.27 1.27)) (justify left))
     )
-    (property "Value" "NJFET" (at 128.27 101.6 0)
+    (property "Value" "J201" (at 128.27 101.6 0)
       (effects (font (size 1.27 1.27)) (justify left))
     )
-    (property "Footprint" "Package_TO_SOT_SMD:SOT-23" (at 128.27 97.79 0)
+    (property "Footprint" "Package_TO_SOT_SMD:SOT-23-3" (at 128.27 97.79 0)
       (effects (font (size 1.27 1.27)) hide)
     )
